File: Frame Strain Gauge.kicad_pcb (KiCad board)
At the start: 4 copper layers, 64 x 20 mm, 93 parts, among them J4 CAN Header, J5 Strain Gauge 3 (Shear), J6 Strain Gauge 2 (Torsion), J7 Strain Gauge 1 (Axial Load), J9 Conn_02x12_Odd_Even, U1 CSTNE8M00GH5C000R0, U2 LSM6DSOXTR, U3 IIS3DWBTR, U4 ADS124S08IPBSR, U5 TPS7A2633DRVR, U6 TCAN332GDR, U8 TPS7A2633DRVR, U9 STM32F412ZGJ6TR

Commit message: prog
Parts:
- removed FL1: Common Mode Choke, Inductor_SMD:L_CommonModeChoke_Coilcraft_0603USB
- added U7: ACT1210-510-2P-TL00, Frame Strain Gauge:CHOKE_10-2P-TL00_TDK, F.Cu at (117.8, 49.5)
- C1, C10, C11, C12, C13, C14, C15, C16, C17, C18, C19, C2, C20, C21, C22, C23, C24, C25, C26, C27, C28, C29, C3, C30, C31, C32, C33, C34, C35, C36, C37, C38, C39, C4, C40, C41, C42, C43, C44, C5, C6, C7, C8, C9: footprint Capacitor_SMD:C_0201_0603Metric -> Capacitor_SMD:C_0603_1608Metric
- C45: footprint Capacitor_SMD:C_0201_0603Metric -> Capacitor_SMD:C_0805_2012Metric
- D1, D2, D3: footprint LED_SMD:LED_0201_0603Metric -> LED_SMD:LED_0603_1608Metric
- D4, D5: footprint Diode_SMD:D_0201_0603Metric -> Diode_SMD:D_SOD-523
- D6: footprint Diode_SMD:D_0201_0603Metric -> Diode_SMD:D_SOD-123
- R1, R10, R17, R18, R19, R2, R20, R21, R22, R23, R24, R25, R26, R27, R28, R3, R4, R5, R6, R7, R8, R9: footprint Resistor_SMD:R_0201_0603Metric -> Resistor_SMD:R_0603_1608Metric
- R11, R12, R13, R14, R15, R16: footprint Resistor_SMD:R_0201_0603Metric -> Resistor_SMD:R_0805_2012Metric
- moved U9 53.3 mm to (92.9, 100.7)
- moved C42 51.6 mm to (122.9, 46.8), turned to 90 degrees
- moved C1 49.3 mm to (127.1, 81.2), turned to -90 degrees
- moved C2 46.8 mm to (124.8, 82.0)
- moved C41 46.0 mm to (121.8, 52.0)
- moved C40 44.0 mm to (122.7, 54.7), turned to -90 degrees
- moved R27 39.2 mm to (121.8, 50.5), turned to 180 degrees
- moved R26 39.0 mm to (121.8, 49.0)
- moved R5 38.1 mm to (127.2, 78.2), turned to 90 degrees
- moved C4 37.4 mm to (115.9, 82.3), turned to -90 degrees
- moved U2 35.9 mm to (113.3, 80.8)
- moved C3 35.8 mm to (113.6, 83.1)
- moved U3 34.7 mm to (124.7, 79.7)
- moved D5 32.9 mm to (120.7, 54.0)
- moved D4 32.0 mm to (118.9, 51.7), turned to 180 degrees
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Routing:
- net GND: track 0.00 -> 22.6 mm, vias 0 -> 8
- net /CANH: track 0.00 -> 11.2 mm
- net /CANL: track 0.00 -> 11.0 mm, vias 0 -> 1
- net +3V3: track 0.00 -> 9.56 mm, vias 0 -> 16
- net Net-(U6-CANH): track 0.00 -> 6.85 mm
- net Net-(U6-CANL): track 0.00 -> 6.74 mm
- net Net-(C42-Pad1): track 0.00 -> 3.11 mm
- net /CS2 LSM6DSOXTR: track 0.00 -> 2.66 mm
- net /CS1 IIS3DWBTR: track 0.00 -> 2.62 mm

Commit message: layout
Parts:
- removed C20, C21, C22, C23, C24, C25, C26, C27, C28, C29, C30, C39: 100 nF, Capacitor_SMD:C_0603_1608Metric
- removed C32: 2.2 uF, Capacitor_SMD:C_0603_1608Metric
- removed J9: Conn_02x12_Odd_Even, Connector_PinHeader_2.00mm:PinHeader_2x12_P2.00mm_Vertical
- removed R3, R4: 4.7k, Resistor_SMD:R_0603_1608Metric
- removed U9: STM32F412ZGJ6TR, Frame Strain Gauge:UFBGA144-10x10mm
- added C46: 100 nF, Capacitor_SMD:C_0603_1608Metric, F.Cu at (94.5, 42.5)
- added C47: 100 nF, Capacitor_SMD:C_0603_1608Metric, F.Cu at (106.2, 43.1)
- added C48: 100 nF, Capacitor_SMD:C_0603_1608Metric, F.Cu at (106.0, 55.0)
- added C49: 100 nF, Capacitor_SMD:C_0603_1608Metric, F.Cu at (94.5, 56.0)
- added J1: Conn_01x05_Pin, Connector_PinHeader_2.00mm:PinHeader_1x05_P2.00mm_Vertical, F.Cu at (103.5, 60.0)
- added U10: STM32F412RGT6, Frame Strain Gauge:LQFP64-10x10mm, F.Cu at (100.2, 49.0)
- moved R10 44.8 mm to (83.3, 42.5), turned to 180 degrees
- moved C17 42.7 mm to (116.0, 52.8)
- moved C31 40.6 mm to (93.5, 44.0), turned to 180 degrees
- moved R7 38.6 mm to (91.0, 43.2), turned to -90 degrees
- moved R28 37.5 mm to (83.3, 44.1), turned to 180 degrees
- moved C3 35.8 mm to (110.9, 47.3)
- moved C4 35.8 mm to (113.2, 46.6)
- moved R6 35.8 mm to (113.2, 43.6)
- moved U2 35.8 mm to (110.6, 45.0)
- moved R21 35.6 mm to (86.5, 51.8), turned to 180 degrees
- moved R14 35.5 mm to (73.1, 44.4), turned to -90 degrees
- moved C1 35.3 mm to (112.8, 48.9), turned to 0 degrees
- moved R13 35.1 mm to (71.2, 44.3), turned to -90 degrees
- moved R19 35.1 mm to (86.5, 48.7), turned to 180 degrees
- moved R18 34.9 mm to (86.5, 47.2), turned to 180 degrees
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Routing:
- net GND: track 22.6 -> 75.8 mm, vias 8 -> 31
- net +5V: track 0.00 -> 40.5 mm, vias 0 -> 2
- net /SPI 1 SCK: track 0.00 -> 33.4 mm, vias 0 -> 3
- net /SPI 1 MOSI: track 0.00 -> 30.2 mm, vias 0 -> 4
- net /SPI 1 MISO: track 0.00 -> 30.0 mm, vias 0 -> 3
- net +3V3: track 9.56 -> 35.1 mm, vias 16 -> 8
- net /MCO: track 0.00 -> 24.5 mm, vias 0 -> 2
- net /SPI 2 SCK: track 0.00 -> 23.3 mm, vias 0 -> 2
- net /SPI 2 MOSI: track 0.00 -> 22.7 mm, vias 0 -> 2
- net /SPI 2 MISO: track 0.00 -> 21.2 mm, vias 0 -> 2
- net /CS3 ADS124S08IPBSR: track 0.00 -> 20.8 mm, vias 0 -> 2
- net /INT LSM6DSOXTR: track 0.00 -> 19.0 mm, vias 0 -> 2
- net /Reset ADS124S08IPBSR: track 0.00 -> 17.3 mm, vias 0 -> 2
- net Net-(U4-AIN2): track 0.00 -> 16.0 mm
- net /Start/Sync ADS124S08IPBSR: track 0.00 -> 15.9 mm
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
Commit message: Completed DRC
Parts:
- moved C19 46.3 mm to (113.3, 43.4), turned to 90 degrees
- moved C18 39.7 mm to (115.9, 56.7)
- moved C33 33.8 mm to (104.8, 57.6)
- moved C37 27.1 mm to (109.6, 57.7)
- moved D1 23.9 mm to (95.1, 58.0)
- moved C38 23.5 mm to (91.8, 45.5), turned to 180 degrees
- moved R25 22.8 mm to (95.1, 59.5)
- moved R8 20.0 mm to (99.6, 56.6)
- moved R24 9.87 mm to (99.6, 58.1)
- moved D2 5.21 mm to (99.6, 59.8), turned to 180 degrees
- moved R6 3.25 mm to (110.2, 42.3), turned to 0 degrees
- moved D3 2.09 mm to (121.1, 58.2)
- moved R23 2.09 mm to (121.1, 59.7)
- moved C49 2.00 mm to (92.5, 56.0)
- moved C34 1.05 mm to (90.6, 52.5)
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Connections:
- R25 pad 1: Net-(U10A-PB9) -> Net-(U10A-PA2)
- U10 pad 16: unconnected-(U10A-PA2-Pad16) -> Net-(U10A-PA2)
- U10 pad 62: Net-(U10A-PB9) -> unconnected-(U10A-PB9-Pad62)
- U5 pad V: (no net) -> GND
- U8 pad V: (no net) -> GND
Routing:
- net +3V3: track 35.1 -> 73.0 mm, vias 8 -> 16
- net /NRST: track 0.00 -> 23.2 mm, vias 0 -> 2
- net /SWCLK: track 0.00 -> 21.2 mm, vias 0 -> 3
- net /SWDIO: track 0.00 -> 17.0 mm, vias 0 -> 1
- net GND: track 75.8 -> 89.4 mm, vias 31 -> 40
- net Net-(U10A-PA2): track 0.00 -> 10.3 mm, vias 0 -> 2
- net Net-(U10A-PB10): track 0.00 -> 4.30 mm
- net +3V3A: track 6.49 -> 9.79 mm, vias 1 -> 3
- net Net-(U10B-VCAP_1): track 0.00 -> 3.29 mm
- net Net-(U10A-PB2): track 0.00 -> 2.91 mm
- net /CAN TXD: track 10.9 -> 13.8 mm
- net Net-(D2-A): track 0.00 -> 1.67 mm
- net /CS1 IIS3DWBTR: track 14.8 -> 16.4 mm
- net /Resonator Output: track 3.99 -> 4.81 mm
- net /DRDY ADS124S08IPBSR: track 14.1 -> 14.8 mm
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- added copper zone on In2.Cu, net +3V3
- added copper zone on In2.Cu, net +3V3A
- added copper zone on B.Cu, net GND
- added copper zone on F.Cu, net GND
- added copper zone on In1.Cu, net GND
Other:
- board text added: "Olin Baja 2026 Designed By Jade Vincent"
