File: Frame Strain Gauge.kicad_sch (KiCad schematic)
At the start: 93 parts, among them J4 CAN Header, J5 Strain Gauge 3 (Shear), J6 Strain Gauge 2 (Torsion), J7 Strain Gauge 1 (Axial Load), J9 Conn_02x12_Odd_Even, U1 CSTNE8M00GH5C000R0, U2 LSM6DSOXTR, U3 IIS3DWBTR, U4 ADS124S08IPBSR, U5 TPS7A2633DRVR, U6 TCAN332GDR, U8 TPS7A2633DRVR, U9 STM32F412ZGJ6TR

Commit message: prog
Parts:
- removed FL1: Common Mode Choke, Inductor_SMD:L_CommonModeChoke_Coilcraft_0603USB, symbol Filter:Choke_CommonMode_FerriteCore_1234
- added U7: ACT1210-510-2P-TL00, Frame Strain Gauge:CHOKE_10-2P-TL00_TDK, symbol Frame Strain Gauge:ACT1210-510-2P-TL00
- C1, C10, C11, C12, C13, C14, C15, C16, C17, C18, C19, C2, C20, C21, C22, C23, C24, C25, C26, C27, C28, C29, C3, C30, C31, C32, C33, C34, C35, C36, C37, C38, C39, C4, C40, C41, C42, C43, C44, C5, C6, C7, C8, C9: footprint Capacitor_SMD:C_0201_0603Metric -> Capacitor_SMD:C_0603_1608Metric
- C45: footprint Capacitor_SMD:C_0201_0603Metric -> Capacitor_SMD:C_0805_2012Metric
- D1, D2, D3: footprint LED_SMD:LED_0201_0603Metric -> LED_SMD:LED_0603_1608Metric
- D4, D5: footprint Diode_SMD:D_0201_0603Metric -> Diode_SMD:D_SOD-523
- D6: footprint Diode_SMD:D_0201_0603Metric -> Diode_SMD:D_SOD-123
- R1, R10, R17, R18, R19, R2, R20, R21, R22, R23, R24, R25, R26, R27, R28, R3, R4, R5, R6, R7, R8, R9: footprint Resistor_SMD:R_0201_0603Metric -> Resistor_SMD:R_0603_1608Metric
- R11, R12, R13, R14, R15, R16: footprint Resistor_SMD:R_0201_0603Metric -> Resistor_SMD:R_0805_2012Metric
Connections:
- net CANH: now also U7.4
- net CANL: now also U7.3
- net at U6.6 (CANL): now also U7.2
- net at U6.7 (CANH): now also U7.1
Other:
- moved on the sheet: C19, C40, C41, C42, D4, D5, R26, R27, U6

Commit message: layout
Parts:
- removed C20, C21, C22, C23, C24, C25, C26, C27, C28, C29, C30, C39: 100 nF, Capacitor_SMD:C_0603_1608Metric, symbol Device:C
- removed C32: 2.2 uF, Capacitor_SMD:C_0603_1608Metric, symbol Device:C
- removed J9: Conn_02x12_Odd_Even, Connector_PinHeader_2.00mm:PinHeader_2x12_P2.00mm_Vertical, symbol Connector_Generic:Conn_02x12_Odd_Even
- removed R3, R4: 4.7k, Resistor_SMD:R_0603_1608Metric, symbol Device:R
- removed U9: STM32F412ZGJ6TR, Frame Strain Gauge:UFBGA144-10x10mm, symbol Frame Strain Gauge:STM32F412ZGJ6TR
- added C46, C47, C48, C49: 100 nF, Capacitor_SMD:C_0603_1608Metric, symbol Device:C
- added J1: Conn_01x05_Pin, Connector_PinHeader_2.00mm:PinHeader_1x05_P2.00mm_Vertical, symbol Connector:Conn_01x05_Pin
- added U10: STM32F412RGT6, Frame Strain Gauge:LQFP64-10x10mm, symbol Frame Strain Gauge:STM32F412RGT6
Connections:
- net +3V3: now also C46.1, C47.1, C48.1, C49.1, J1.1 (Pin_1), U10.1 (VBAT), U10.13 (VDDA/VREF+), U10.19 (VDD), U10.32 (VDD), U10.48 (VDD), U10.64 (VDD)
- net CAN RXD: now also U10.44 (PA11)
- net CAN TXD: now also U10.45 (PA12)
- net CS1 IIS3DWBTR: now also U10.55 (PB3)
- net CS2 LSM6DSOXTR: now also U10.56 (PB4)
- net CS3 ADS124S08IPBSR: now also U10.57 (PB5)
- net DRDY ADS124S08IPBSR: now also U10.17 (PA3)
- net GND: now also C46.2, C47.2, C48.2, C49.2, J1.5 (Pin_5), U10.12 (VSSA/VREF-), U10.18 (VSS), U10.31 (VSS), U10.47 (VSS), U10.63 (VSS)
- net INT IIS3DWBTR: now also U10.26 (PB0)
- net INT LSM6DSOXTR: now also U10.27 (PB1)
- net MCO: now also U10.40 (PC9)
- net NRST: now also J1.4 (Pin_4), U10.7 (NRST)
- net Reset ADS124S08IPBSR: now also U10.61 (PB8)
- net Resonator Input: now also U10.5 (PH0-OSC_IN)
- net Resonator Output: now also U10.6 (PH1)
- net SPI 1 MISO: now also U10.22 (PA6)
- net SPI 1 MOSI: now also U10.23 (PA7)
- net SPI 1 SCK: now also U10.21 (PA5)
- net SPI 2 MISO: now also U10.35 (PB14)
- net SPI 2 MOSI: now also U10.36 (PB15)
- net SPI 2 SCK: now also U10.34 (PB13)
- net SWCLK: now also J1.2 (Pin_2), U10.49 (PA14)
- net SWDIO: now also J1.3 (Pin_3), U10.46 (PA13)
- net Start/Sync ADS124S08IPBSR: now also U10.20 (PA4)
- net at R25.1: now also U10.62 (PB9)
- net at R8.2: now also U10.28 (PB2)
- net at R24.2: now also U10.29 (PB10)
- net at C33.1: now also U10.30 (VCAP_1)
- net at R7.1: now also U10.60 (BOOT0)
Other:
- moved on the sheet: C1, C10, C11, C12, C13, C14, C15, C16, C17, C18, C19, C2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

Commit message: Completed DRC
Connections:
- net at R25.1: now also U10.16 (PA2); no longer U10.62 (PB9)
